File: panels/pcb/10hp_generic/10hp_generic.sch (KiCad schematic (older format))
At the start: 81 parts, among them J1 Conn_02x04_Odd_Even, J2 SWD, SW1 SW_Push, SW10 SW_Push, SW11 SW_Push, SW12 SW_Push, SW13 SW_Push, SW14 SW_Push, SW15 SW_Push, SW16 SW_Push, SW2 SW_Push, SW3 SW_Push, SW4 SW_Push, SW5 SW_Push, SW6 SW_Push, SW7 SW_Push, SW8 SW_Push, SW9 SW_Push, U1 STM32F072RBTx, U2 AMS1117-3.3

Commit message: Fixes PCB footprint for C27 & C29
Parts:
- C27, C29: LCSC C2918489 -> C5252390
Changed lines of the file:
@@
 F 2 "Capacitor_SMD:C_0402_1005Metric" H 5488 4900 50  0001 C CNN
 F 3 "~" H 5450 5050 50  0001 C CNN
-F 4 "C2918489" H 5450 5050 50  0001 C CNN "LCSC"
+F 4 "C5252390" H 5450 5050 50  0001 C CNN "LCSC"
 	1    5450 5050
 	1    0    0    -1
@@
 F 2 "Capacitor_SMD:C_0402_1005Metric" H 6388 4900 50  0001 C CNN
 F 3 "~" H 6350 5050 50  0001 C CNN
-F 4 "C2918489" H 6350 5050 50  0001 C CNN "LCSC"
+F 4 "C5252390" H 6350 5050 50  0001 C CNN "LCSC"
 	1    6350 5050
 	1    0    0    -1

Commit message: Fixes some component values
Parts:
- C32, C34: LCSC C2918489 -> C5137476
Changed lines of the file:
@@
 F 2 "Capacitor_SMD:C_0805_2012Metric" H 10388 5800 50  0001 C CNN
 F 3 "~" H 10350 5950 50  0001 C CNN
-F 4 "C2918489" H 10350 5950 50  0001 C CNN "LCSC"
+F 4 "C5137476" H 10350 5950 50  0001 C CNN "LCSC"
 	1    10350 5950
 	1    0    0    -1
@@
 F 2 "Capacitor_SMD:C_0805_2012Metric" H 9038 5800 50  0001 C CNN
 F 3 "~" H 9000 5950 50  0001 C CNN
-F 4 "C2918489" H 9000 5950 50  0001 C CNN "LCSC"
+F 4 "C5137476" H 9000 5950 50  0001 C CNN "LCSC"
 	1    9000 5950
 	1    0    0    -1

Commit message: R2 of generic PCB using different components
Parts:
- removed D1: WS2812B, WS2812:XL-3528RGBW-WS2812B, symbol LED:WS2812B
- added D1: WS2812B, WS2812:XL-2121RGBC-WS2812B, symbol WS2812:XL-2121RGBC-WS2812B
- C1, C10, C11, C12, C13, C14, C15, C16, C17, C18, C19, C2, C20, C21, C22, C23, C24, C25, C26, C28, C3, C33, C35, C36, C37, C4, C5, C6, C7, C8, C9: LCSC C392963 -> C1525
- C27, C29: footprint Capacitor_SMD:C_0402_1005Metric -> Capacitor_SMD:C_0805_2012Metric; LCSC C5252390 -> C1779
- C30: LCSC C1524 -> C15195
- C31: LCSC C164868 -> C52923
- C32, C34: LCSC C5137476 -> C15850
- D10, D11, D12, D13, D14, D15, D16, D2, D3, D4, D5, D6, D7, D8, D9: footprint WS2812:XL-3528RGBW-WS2812B -> WS2812:XL-2121RGBC-WS2812B; symbol LED:WS2812B -> WS2812:XL-2121RGBC-WS2812B; LCSC C2890364 -> C5349957
- SW13: LCSC (none) -> C5260475
- U2: LCSC C5181460 -> C6186
Connections:
- net +5V: now also D10.3 (VDD), D11.3 (VDD), D12.3 (VDD), D13.3 (VDD), D14.3 (VDD), D15.3 (VDD), D16.3 (VDD), D2.3 (VDD), D3.3 (VDD), D4.3 (VDD), D5.3 (VDD), D6.3 (VDD), D7.3 (VDD), D8.3 (VDD), D9.3 (VDD), D1.3 (VDD); no longer D10.1 (VDD), D11.1 (VDD), D12.1 (VDD), D13.1 (VDD), D14.1 (VDD), D15.1 (VDD), D16.1 (VDD), D2.1 (VDD), D3.1 (VDD), D4.1 (VDD), D5.1 (VDD), D6.1 (VDD), D7.1 (VDD), D8.1 (VDD), D9.1 (VDD)
- net GND: now also D10.1 (VSS), D11.1 (VSS), D12.1 (VSS), D13.1 (VSS), D14.1 (VSS), D15.1 (VSS), D16.1 (VSS), D2.1 (VSS), D3.1 (VSS), D4.1 (VSS), D5.1 (VSS), D6.1 (VSS), D7.1 (VSS), D8.1 (VSS), D9.1 (VSS), D1.1 (VSS); no longer D10.3 (VSS), D11.3 (VSS), D12.3 (VSS), D13.3 (VSS), D14.3 (VSS), D15.3 (VSS), D16.3 (VSS), D2.3 (VSS), D3.3 (VSS), D4.3 (VSS), D5.3 (VSS), D6.3 (VSS), D7.3 (VSS), D8.3 (VSS), D9.3 (VSS)
- net WS2812: now also D1.2 (DIN)
- net at D2.4 (DOUT): now also D3.2 (DIN)
- net at D2.2 (DIN): now also D1.4 (DOUT); no longer D3.4 (DIN)
- net at D4.4 (DOUT): now also D5.2 (DIN); no longer D3.2 (DOUT)
- net at D4.2 (DIN): now also D3.4 (DOUT); no longer D5.4 (DIN)
- net at D6.4 (DOUT): now also D7.2 (DIN); no longer D5.2 (DOUT)
- net at D6.2 (DIN): now also D5.4 (DOUT); no longer D7.4 (DIN)
- net at D8.4 (DOUT): now also D9.2 (DIN); no longer D7.2 (DOUT)
- net at D8.2 (DIN): now also D7.4 (DOUT); no longer D9.4 (DIN)
- net at D10.4 (DOUT): now also D11.2 (DIN); no longer D9.2 (DOUT)
- net at D10.2 (DIN): now also D9.4 (DOUT); no longer D11.4 (DIN)
- net at D12.4 (DOUT): now also D13.2 (DIN); no longer D11.2 (DOUT)
- net at D12.2 (DIN): now also D11.4 (DOUT); no longer D13.4 (DIN)
- net at D14.4 (DOUT): now also D15.2 (DIN); no longer D13.2 (DOUT)
- net at D14.2 (DIN): now also D13.4 (DOUT); no longer D15.4 (DIN)
- net at D16.4 (DOUT): no longer D15.2 (DOUT)
- net at D16.2 (DIN): now also D15.4 (DOUT)
